File: bass_big_muff2.kicad_pcb (KiCad board)
At the start: 2 copper layers, 60.3 x 101 mm, 93 parts, among them SW1 SW_DPDT_x3, SW2 SW_DPDT_x2, U1 TL074, U2 TL074

Commit message: V2
Parts:
- removed C19: 4n7, Capacitor_THT:C_Rect_L7.2mm_W2.5mm_P5.00mm
- removed R26: 4k7, Resistor_THT:R_Axial_DIN0207_L6.3mm_D2.5mm_P7.62mm_Horizontal
- removed REF**: 1590N1_125B, enclosures:1590N1_125B
- C15, C21, C23, C24, C8: value 100n -> 220n
- C18: value 22n -> 4n7
- R35: value 10k -> 33k
- SUSTAIN1, TONE1, VOLUME1: moved to B.Cu
- moved C1 17.2 mm to (137.8, 76.9), turned to 180 degrees
- moved VOLUME1 10.4 mm to (167.8, 65.4), turned to 180 degrees
- moved TONE1 10.0 mm to (147.0, 69.9), turned to 180 degrees
- moved SUSTAIN1 10.0 mm to (126.7, 65.4), turned to 180 degrees
- moved C20 6.23 mm to (139.1, 85.3)
- moved C22 6.23 mm to (139.1, 82.1)
Connections:
- C11 pad 1: Net-(U2A--) -> Net-(U2A-+)
- C20 pad 1: Net-(C19-Pad1) -> Net-(D10-K)
- C5 pad 1: Net-(U1A--) -> Net-(U1A-+)
- PAD6 pad 1: Net-(SW1B-B) -> Net-(SW1B-A)
- R14 pad 2: Net-(U2A--) -> Net-(U2A-+)
- R27 pad 1: Net-(C19-Pad1) -> Net-(D10-K)
- R29 pad 1: Net-(C19-Pad1) -> Net-(D10-K)
- R3 pad 2: Net-(U1A--) -> Net-(U1A-+)
- R4 pad 1: Net-(U1A--) -> Net-(U1A-+)
- R5 pad 2: Net-(U1A-+) -> Net-(U1A--)
- SW1 pad 4: Net-(SW1B-B) -> Net-(D2-K)
- SW1 pad 5: Net-(D2-K) -> Net-(SW1B-A)
- U2 pad 2: Net-(U2A--) -> Net-(D7-K)
- U2 pad 3: Net-(D7-K) -> Net-(U2A-+)
Routing:
- net Net-(D10-K): track 14.4 -> 70.1 mm
- net Net-(C19-Pad1): track 53.4 -> 0.00 mm
- net Net-(SW1A-A): track 23.9 -> 7.30 mm
- net GND: track 285.4 -> 270.2 mm
- net Net-(D2-K): track 14.1 -> 0.00 mm
- net VCC: track 122.6 -> 108.8 mm
- net Net-(SW2B-C): track 10.5 -> 22.0 mm
- net Net-(SW2B-B): track 121.5 -> 110.9 mm
- net Net-(C21-Pad1): track 12.4 -> 21.2 mm
- net Net-(SW1B-B): track 7.98 -> 0.00 mm
- net Net-(U2A-+): track 0.00 -> 7.00 mm
- net Net-(U2A--): track 6.59 -> 0.00 mm
- net Net-(R35-Pad2): track 73.4 -> 68.4 mm
- net Net-(D7-K): track 24.9 -> 27.9 mm
- net Net-(C21-Pad2): track 23.1 -> 24.8 mm
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