File: bass_big_muff2.kicad_sch (KiCad schematic)
At the start: 92 parts, among them SW1 SW_DPDT_x3, SW2 SW_DPDT_x2, U1 TL074, U2 TL074

Commit message: V2
Parts:
- removed C19: 4n7, Capacitor_THT:C_Rect_L7.2mm_W2.5mm_P5.00mm, symbol Device:C
- removed R26: 4k7, Resistor_THT:R_Axial_DIN0207_L6.3mm_D2.5mm_P7.62mm_Horizontal, symbol Device:R
- C15, C21, C23, C24, C8: value 100n -> 220n
- C18: value 22n -> 4n7
- R35: value 10k -> 33k
Connections:
- net at C5.1, R3.2, R4.1: now also U1.3 (+); no longer U1.2 (-)
- net at C17.2, D10.1 (K), D9.2 (A)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: now also C20.1, R27.1, R29.1
- net at C13.1, D7.1 (K), D8.2 (A)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: now also U2.2 (-); no longer U2.3 (+)
- net at R5.2: now also U1.2 (-); no longer U1.3 (+)
- net at PAD6.1: now also SW1.5 (B); no longer SW1.4 (B)
- net at C11.1, R14.2: now also U2.3 (+); no longer U2.2 (-)
- net at D2.1 (K): now also SW1.4 (A); no longer SW1.5 (A)
Other:
- note removed: "NOTES TO SELF: - I messed up the DPDT switch footprint's pin numbering - a few B.Cu traces need some attention. Especially towards the board edge - also 3PDT wiring is messed up. pins 4 and 5 are switched up - change coupling cap values to align with reality - audioprobe leg 1 of C24 - you flipped an op-amp dumbass (U2A) - C18 should be way smaller (e.g. 4n7) - Test if bridging R26 solves low out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"
- moved on the sheet: BASS_CTRL1, C18, C20, C21, C22, C23, C24, C25, R27, R28, R29, R30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
